Commit message: basic framework

File: src/GigaVacuumMobil/urdf/GigaVacuumMobile.urdf.xacro (robot description, xacro)
@@ -1,7 +1,9 @@
 <?xml version="1.0"?>
 <robot xmlns:xacro="http://www.ros.org/wiki/xacro" name="GigaVacuumMobil">
+    <!-- ============ ADD THIS ARGUMENT AT THE TOP ============ -->
+    <xacro:arg name="use_sim" default="false"/>
     <!-- Robot constants - UPDATE THESE TO MATCH YOUR ACTUAL ROBOT -->
-    <xacro:property name="wheel_radius" value="0.033" /> <!-- 3.3 cm -->
-    <xacro:property name="wheel_separation" value="0.17" /> <!-- 17 cm between wheels -->
+    <xacro:property name="wheel_radius" value="0.033" />
+    <xacro:property name="wheel_separation" value="0.17" />
     <xacro:property name="wheel_width" value="0.02" />
     <xacro:property name="base_length" value="0.20" />
@@ -26,4 +28,8 @@
             </geometry>
         </collision>
+        <inertial>
+            <mass value="1.0"/>
+            <inertia ixx="0.001" ixy="0.0" ixz="0.0" iyy="0.001" iyz="0.0" izz="0.001"/>
+        </inertial>
     </link>
     <!-- Right Wheel -->
@@ -44,4 +50,8 @@
             <origin xyz="0 0 0" rpy="1.5707 0 0" />
         </collision>
+        <inertial>
+            <mass value="0.1"/>
+            <inertia ixx="0.0001" ixy="0.0" ixz="0.0" iyy="0.0001" iyz="0.0" izz="0.0001"/>
+        </inertial>
     </link>
     <joint name="right_wheel_joint" type="continuous">
@@ -66,4 +76,8 @@
             <origin xyz="0 0 0" rpy="1.5707 0 0" />
         </collision>
+        <inertial>
+            <mass value="0.1"/>
+            <inertia ixx="0.0001" ixy="0.0" ixz="0.0" iyy="0.0001" iyz="0.0" izz="0.0001"/>
+        </inertial>
     </link>
     <joint name="left_wheel_joint" type="continuous">
@@ -83,4 +97,8 @@
             </material>
         </visual>
+        <inertial>
+            <mass value="0.1"/>
+            <inertia ixx="0.0001" ixy="0.0" ixz="0.0" iyy="0.0001" iyz="0.0" izz="0.0001"/>
+        </inertial>
     </link>
     <joint name="lidar_joint" type="fixed">
@@ -95,9 +113,10 @@
         <hardware>
             <plugin>GigaVacuumMobil/DiffDriveHardware</plugin>
-            <!-- Parameters for your hardware interface -->
+            <!-- ============ MODIFIED: Conditional fake_hardware parameter ============ -->
+            <param name="fake_hardware">$(arg use_sim)</param>
             <param name="device">/dev/ttyUSB0</param>
             <param name="baud_rate">57600</param>
             <param name="timeout_ms">100</param>
-            <param name="enc_ticks_per_rev">2400</param> <!-- UPDATE THIS! -->
+            <param name="enc_ticks_per_rev">2400</param>
         </hardware>
         <!-- Define the joints that this hardware interface controls -->

Commit message: sim working with slam. navigation started

File: src/GigaVacuumMobil/urdf/GigaVacuumMobile.urdf.xacro (robot description, xacro)
@@ -3,8 +3,10 @@
     <!-- ============ ADD THIS ARGUMENT AT THE TOP ============ -->
     <xacro:arg name="use_sim" default="false"/>
+    <xacro:arg name="controllers_file" default=""/>
     <!-- Robot constants - UPDATE THESE TO MATCH YOUR ACTUAL ROBOT -->
     <xacro:property name="wheel_radius" value="0.033" />
     <xacro:property name="wheel_separation" value="0.17" />
     <xacro:property name="wheel_width" value="0.02" />
+    <xacro:property name="wheel_offset_x" value="0.04" />
     <xacro:property name="base_length" value="0.20" />
     <xacro:property name="base_width" value="0.15" />
@@ -52,5 +54,6 @@
         <inertial>
             <mass value="0.1"/>
-            <inertia ixx="0.0001" ixy="0.0" ixz="0.0" iyy="0.0001" iyz="0.0" izz="0.0001"/>
+            <origin xyz="0 0 0" rpy="1.5707 0 0" />
+            <inertia ixx="0.00005" ixy="0.0" ixz="0.0" iyy="0.00005" iyz="0.0" izz="0.00005"/>
         </inertial>
     </link>
@@ -58,5 +61,5 @@
         <parent link="base_link" />
         <child link="right_wheel_link" />
-        <origin xyz="0 ${-wheel_separation/2} 0" rpy="0 0 0" />
+        <origin xyz="${wheel_offset_x} ${-wheel_separation/2} 0" rpy="0 0 0" />
         <axis xyz="0 1 0" />
     </joint>
@@ -78,5 +81,6 @@
         <inertial>
             <mass value="0.1"/>
-            <inertia ixx="0.0001" ixy="0.0" ixz="0.0" iyy="0.0001" iyz="0.0" izz="0.0001"/>
+            <origin xyz="0 0 0" rpy="1.5707 0 0" />
+            <inertia ixx="0.00005" ixy="0.0" ixz="0.0" iyy="0.00005" iyz="0.0" izz="0.00005"/>
         </inertial>
     </link>
@@ -84,6 +88,33 @@
         <parent link="base_link" />
         <child link="left_wheel_link" />
-        <origin xyz="0 ${wheel_separation/2} 0" rpy="0 0 0" />
+        <origin xyz="${wheel_offset_x} ${wheel_separation/2} 0" rpy="0 0 0" />
         <axis xyz="0 1 0" />
+    </joint>
+    <!-- Caster Wheel (Pivot/Support Wheel) -->
+    <xacro:property name="caster_radius" value="0.015" />
+    <xacro:property name="caster_offset_x" value="${-base_length/2 + 0.02}" />
+    <link name="caster_wheel_link">
+        <visual>
+            <geometry>
+                <sphere radius="${caster_radius}" />
+            </geometry>
+            <material name="gray">
+                <color rgba="0.5 0.5 0.5 1.0" />
+            </material>
+        </visual>
+        <collision>
+            <geometry>
+                <sphere radius="${caster_radius}" />
+            </geometry>
+        </collision>
+        <inertial>
+            <mass value="0.05"/>
+            <inertia ixx="0.00001" ixy="0.0" ixz="0.0" iyy="0.00001" iyz="0.0" izz="0.00001"/>
+        </inertial>
+    </link>
+    <joint name="caster_wheel_joint" type="fixed">
+        <parent link="base_link" />
+        <child link="caster_wheel_link" />
+        <origin xyz="${caster_offset_x} 0 ${-wheel_radius + caster_radius}" rpy="0 0 0" />
     </joint>
     <!-- Lidar Sensor (RPLIDAR C1) -->
@@ -97,4 +128,9 @@
             </material>
         </visual>
+        <collision>
+            <geometry>
+                <cylinder radius="0.05" length="0.04"/>
+            </geometry>
+        </collision>
         <inertial>
             <mass value="0.1"/>
@@ -107,4 +143,34 @@
         <origin xyz="${lidar_offset_x} 0 ${lidar_offset_z}" rpy="0 0 0" />
     </joint>
+    <!-- Gazebo Lidar Sensor Plugin -->
+    <gazebo reference="lidar_link">
+        <sensor name="lidar_sensor" type="gpu_lidar">
+            <topic>scan</topic>
+            <update_rate>10</update_rate>
+            <gz_frame_id>lidar_link</gz_frame_id>
+            <lidar>
+                <scan>
+                    <horizontal>
+                        <samples>360</samples>
+                        <resolution>1</resolution>
+                        <min_angle>0.0</min_angle>
+                        <max_angle>6.28</max_angle>
+                    </horizontal>
+                </scan>
+                <range>
+                    <min>0.12</min>
+                    <max>12.0</max>
+                    <resolution>0.01</resolution>
+                </range>
+                <noise>
+                    <type>gaussian</type>
+                    <mean>0.0</mean>
+                    <stddev>0.01</stddev>
+                </noise>
+            </lidar>
+            <always_on>1</always_on>
+            <visualize>true</visualize>
+        </sensor>
+    </gazebo>
     <!-- =================================================================== -->
     <!-- |                      ROS2 Control Plugin                        | -->
@@ -112,11 +178,15 @@
     <ros2_control name="GigaVacuumMobil" type="system">
         <hardware>
-            <plugin>GigaVacuumMobil/DiffDriveHardware</plugin>
-            <!-- ============ MODIFIED: Conditional fake_hardware parameter ============ -->
-            <param name="fake_hardware">$(arg use_sim)</param>
-            <param name="device">/dev/ttyUSB0</param>
-            <param name="baud_rate">57600</param>
-            <param name="timeout_ms">100</param>
-            <param name="enc_ticks_per_rev">2400</param>
+            <!-- Use different plugin based on simulation mode -->
+            <xacro:if value="$(arg use_sim)">
+                <plugin>gz_ros2_control/GazeboSimSystem</plugin>
+            </xacro:if>
+            <xacro:unless value="$(arg use_sim)">
+                <plugin>GigaVacuumMobil/DiffDriveHardware</plugin>
+                <param name="device">/dev/ttyUSB0</param>
+                <param name="baud_rate">57600</param>
+                <param name="timeout_ms">100</param>
+                <param name="enc_ticks_per_rev">2400</param>
+            </xacro:unless>
         </hardware>
         <!-- Define the joints that this hardware interface controls -->
@@ -132,3 +202,46 @@
         </joint>
     </ros2_control>
+    <!-- Gazebo ros2_control plugin -->
+    <gazebo>
+        <plugin filename="gz_ros2_control-system" name="gz_ros2_control::GazeboSimROS2ControlPlugin">
+            <robot_param>robot_description</robot_param>
+            <robot_param_node>/robot_state_publisher</robot_param_node>
+            <parameters>$(arg controllers_file)</parameters>
+        </plugin>
+    </gazebo>
+    <!-- Gazebo-specific material properties -->
+    <gazebo reference="base_link">
+        <material>Gazebo/Blue</material>
+    </gazebo>
+    <gazebo reference="left_wheel_link">
+        <material>Gazebo/Black</material>
+        <mu1>1.0</mu1>
+        <mu2>1.0</mu2>
+        <kp>1000000.0</kp>
+        <kd>100.0</kd>
+        <minDepth>0.001</minDepth>
+        <maxVel>1.0</maxVel>
+    </gazebo>
+    <gazebo reference="right_wheel_link">
+        <material>Gazebo/Black</material>
+        <mu1>1.0</mu1>
+        <mu2>1.0</mu2>
+        <kp>1000000.0</kp>
+        <kd>100.0</kd>
+        <minDepth>0.001</minDepth>
+        <maxVel>1.0</maxVel>
+    </gazebo>
+    <gazebo reference="caster_wheel_link">
+        <material>Gazebo/Gray</material>
+        <!-- Low friction for smooth pivoting -->
+        <mu1>0.0</mu1>
+        <mu2>0.0</mu2>
+        <kp>1000000.0</kp>
+        <kd>100.0</kd>
+        <minDepth>0.001</minDepth>
+        <maxVel>1.0</maxVel>
+    </gazebo>
+    <gazebo reference="lidar_link">
+        <material>Gazebo/Red</material>
+    </gazebo>
 </robot>
